File: hw/rk86_sd/rk86_sd.kicad_sch (KiCad schematic)
At the start: 16 parts, among them J1 PC Interface, J2 AVR ISP, J3 Micro_SD_Card_Det_Hirose_DM3AT, U1 ATmega328-A, U2 AMS1117-3.3, U3 4050

Commit message: small pcb edition
Parts:
- J2: footprint Connector_PinHeader_2.00mm:PinHeader_2x03_P2.00mm_Vertical -> Connector_PinHeader_2.54mm:PinHeader_2x03_P2.54mm_Vertical
Connections:
- net BUS_A4: now also U1.27 (PC4); no longer U1.28 (PC5)
- net BUS_A5: now also U1.28 (PC5); no longer U1.27 (PC4)
- net BUS_A6: now also U1.7 (XTAL1/PB6); no longer U1.8 (XTAL2/PB7)
- net BUS_A7: now also U1.8 (XTAL2/PB7); no longer U1.7 (XTAL1/PB6)
